Commit message: corrected camera position

File: m2wr_description/urdf/m2wr.xacro (robot description, xacro)
@@ -94,5 +94,5 @@
     <!-- Create camera instance -->
     <xacro:realsense-rs200 prefix="m2wr_" parent="link_chassis">
-        <origin xyz="0 0 1.0" rpy="0 0 0" />
+        <origin xyz="0 0 0.3" rpy="0 0 0" />
     </xacro:realsense-rs200>
 </robot>
